File: hardware/iida_devkit.kicad_pcb (KiCad board)
At the start: 6 copper layers, 227 parts, among them J201 B2B-XH-A, J202 USB4105-GF-A, J203 PRPC001DAAN-RC, J204 PRPC001DAAN-RC, J205 61300111121, J206 61300111121, J207 61300111121, J208 PRPC001DAAN-RC, J209 PRPC001DAAN-RC, J301 TC2050, J302 61300611121, J303 61300611121, J304 61300611121, J305 61300611121, J306 61300611121, J501 SIM8066-6-1-14-01-A, J601 SMA 132134, Q201 IRLML6401, Q202 DMN2005, Q203 DMN2005, Q301 BSS806NH, Q501 BSS806NH, Q502 IRLML6401, Q503 BSS806NH, Q504 BSS806NH, Q505 BSS806NH, Q506 BSS806NH, SW301 PTS645S, SW302 PTS645S, U201 BQ29728DSER, U202 LM66200DRLR, U203 MCP73833T-FCI/MF, U204 TPS63020DSJR, U205 MAX17048G+T10, U301 STM32L552CET6, U401 TCA9554PW, U402 AT25SF081B-MAHB-T, U403 MCP9808T-E/MC, U404 M24256E-B, U405 SHT40-AD1B-R2, U501 TXS0108E, U502 BG770AGLAA-N06-SGNSA, Y301 ECS-160-9-37-CKM-TR3, Y302 ABS05-32.768KHZ-9-T

Commit message: HW: Redo power layout
Parts:
- removed the C505 at (211.6, 102.4)
- removed the D502 at (-86.6, 73.0)
- removed the Q506 at (-116.8, 67.7)
- removed the R314 at (69.0, 140.3)
- removed the R507 at (221.0, 105.0)
- removed the R517 at (201.3, 112.5)
- removed the R522 at (-91.7, 73.7)
- removed the R523 at (-91.7, 75.3)
- removed the R524 at (-89.6, 64.1)
- added C217: 10 µF, Capacitor_SMD:C_0603_1608Metric, F.Cu at (127.4, 69.2)
- added C218: 0.1 µF, perfect_footprints:C_0201_0603Metric, F.Cu at (125.7, 61.3)
- added C219: 10 µF, Capacitor_SMD:C_0603_1608Metric, F.Cu at (127.8, 61.9)
- added C502: 22 µF, Capacitor_SMD:C_0603_1608Metric, F.Cu at (30.6, 20.3)
- added C507: 100 µF, Capacitor_SMD:CP_Elec_6.3x3, F.Cu at (27.7, 3.58)
- added C510: 0.1 µF, perfect_footprints:C_0201_0603Metric, F.Cu at (26.4, 42.6)
- added C511: 0.1 µF, perfect_footprints:C_0201_0603Metric, F.Cu at (23.5, 19.0)
- added C512: 10000 pF, perfect_footprints:C_0201_0603Metric, F.Cu at (26.4, 44.2)
- added C513: 10000 pF, perfect_footprints:C_0201_0603Metric, F.Cu at (23.5, 20.6)
- added C515: 100 pF, perfect_footprints:C_0201_0603Metric, F.Cu at (26.4, 45.8)
- added C516: 100 pF, perfect_footprints:C_0201_0603Metric, F.Cu at (23.5, 22.2)
- added C517: 10000 pF, perfect_footprints:C_0201_0603Metric, F.Cu at (23.5, 23.8)
- added D205: RED, LED_SMD:LED_0603_1608Metric, F.Cu at (132.0, 74.1)
- added D501: RED, LED_SMD:LED_0603_1608Metric, F.Cu at (149.4, 152.3)
- added D504: RED, LED_SMD:LED_0603_1608Metric, F.Cu at (134.4, 152.4)
- added FB502: BLM21BB201SH1D, Inductor_SMD:L_0805_2012Metric, F.Cu at (29.9, 14.2)
- added J205: PRPC001DAAN-RC, Connector_PinHeader_2.54mm:PinHeader_1x02_P2.54mm_Vertical, F.Cu at (106.7, 79.4)
- added J209: PRPC001DAAN-RC, Connector_PinHeader_2.54mm:PinHeader_1x02_P2.54mm_Vertical, F.Cu at (129.4, 72.3)
- added J212: PRPC001DAAN-RC, Connector_PinHeader_2.54mm:PinHeader_1x02_P2.54mm_Vertical, F.Cu at (126.7, 59.2)
- added Q505: BSS806NH, Package_TO_SOT_SMD:SOT-23-3, F.Cu at (152.0, 154.0)
- added Q507: BSS806NH, Package_TO_SOT_SMD:SOT-23-3, F.Cu at (137.0, 154.0)
- added R208: 0 Ω, Resistor_SMD:R_0805_2012Metric, F.Cu at (108.0, 82.2)
- added R215: 2.2 kΩ, perfect_footprints:R_0201_0603Metric, F.Cu at (132.0, 72.0)
- added R221: 1.2 MΩ, perfect_footprints:R_0201_0603Metric, F.Cu at (122.3, 79.9)
- added R223: 1.02 MΩ, perfect_footprints:R_0201_0603Metric, F.Cu at (125.7, 62.7)
- added R224: 180 kΩ, perfect_footprints:R_0201_0603Metric, F.Cu at (125.1, 62.0)
- added R225: 0 Ω, Resistor_SMD:R_0805_2012Metric, F.Cu at (125.7, 56.4)
- added R313: 22 Ω, perfect_footprints:R_0201_0603Metric, F.Cu at (67.8, 141.9)
- added R504: 330 Ω, perfect_footprints:R_0201_0603Metric, F.Cu at (28.4, 45.8)
- added R514: 22 Ω, perfect_footprints:R_0201_0603Metric, F.Cu at (30.5, 41.0)
- added R515: 22 Ω, perfect_footprints:R_0201_0603Metric, F.Cu at (30.5, 42.6)
- added R520: 330 Ω, perfect_footprints:R_0201_0603Metric, F.Cu at (151.1, 156.7)
- added R521: 2.2 kΩ, perfect_footprints:R_0201_0603Metric, F.Cu at (151.7, 151.5)
- added R525: 180 kΩ, perfect_footprints:R_0201_0603Metric, F.Cu at (136.8, 156.7)
- added R527: 330 Ω, perfect_footprints:R_0201_0603Metric, F.Cu at (136.1, 156.7)
- added R529: 2.2 kΩ, perfect_footprints:R_0201_0603Metric, F.Cu at (136.7, 151.6)
- added TP203: TestPoint, TestPoint:TestPoint_Pad_D1.0mm, B.Cu at (126.7, 56.4)
- added U206: LD39200DPUR, Package_DFN_QFN:DFN-8-1EP_4x4mm_P0.8mm_EP2.3x3.24mm, F.Cu at (125.8, 65.7)
- C501: value 100 µF -> 22 µF; footprint Capacitor_SMD:CP_Elec_6.3x3 -> Capacitor_SMD:C_0603_1608Metric
- C504: value 1 µF -> 22 µF; footprint perfect_footprints:C_0201_0603Metric -> Capacitor_SMD:C_0603_1608Metric
- C506: value 10000 pF -> 100 µF; footprint perfect_footprints:C_0201_0603Metric -> Capacitor_SMD:CP_Elec_6.3x3
- C508: value 100 pF -> 1 µF
- C509: value 10000 pF -> 1 µF
- R201, R202: footprint perfect_footprints:R_0402_1005Metric -> perfect_footprints:R_0201_0603Metric
- R213: renamed from R216; value 1.02 MΩ -> 1.2 MΩ
- R509, R510: value 22 Ω -> 330 Ω
- R518: value 22 Ω -> 180 kΩ
- U502: value BG770AGLAA-N06-SGNSA -> BG95M4LA-64-SGNS; footprint Quectel:Quectel_BG77 -> RF_GSM:Quectel_BG95
- moved Q506 276.7 mm to (144.6, 154.0), turned to 90 degrees
- moved R524 251.9 mm to (144.4, 156.7), turned to 90 degrees
- moved R526 250.7 mm to (143.7, 156.7), turned to 90 degrees
- moved R528 249.0 mm to (144.3, 151.5)
- moved D503 242.8 mm to (142.0, 152.3), turned to -90 degrees
- moved Q501 211.4 mm to (22.7, 34.3), turned to 0 degrees
- moved U502 210.8 mm to (11.0, 12.8)
- moved Q502 206.3 mm to (22.7, 38.7), turned to 0 degrees
- moved C501 205.8 mm to (30.6, 17.8), turned to 0 degrees
- moved R502 203.9 mm to (28.4, 42.6), turned to 0 degrees
- moved R501 203.6 mm to (28.4, 41.0), turned to 0 degrees
- moved R503 202.8 mm to (28.4, 44.2), turned to 0 degrees
- moved FB501 201.2 mm to (22.4, 42.3), turned to 0 degrees
- moved C503 199.9 mm to (22.2, 44.9)
- moved C504 199.0 mm to (30.6, 22.8), turned to 0 degrees
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- renumbered C208 to C206, C206 to C207, C207 to C208, C212 to C211, C211 to C212, C214 to C213, C215 to C214, C216 to C215, C213 to C216, C502 to C505, C507 to C514, C510 to C518, C511 to C519, C512 to C520, C513 to C521, D205 to D206, D206 to D207, D207 to D208, D208 to D209, D503 to D502, D501 to D503, J205 to J206, J206 to J207, J207 to J208, J208 to J210, J209 to J211, Q505 to Q506, R205 to R204, R204 to R205, R210 to R209, R211 to R210, R208 to R211, R209 to R212, R217 to R214, R212 to R216, R213 to R217, R214 to R218, R215 to R220, R218 to R222, R313 to R314, R504 to R505, R505 to R506, R511 to R507, R512 to R508, R515 to R511, R506 to R512, R508 to R513, R513 to R517, R514 to R519, R525 to R522, R526 to R523, R519 to R524, R520 to R526, R521 to R528, TP203 to TP204, TP204 to TP205, TP205 to TP206
Connections:
- net /Modem/EN_V_3V3_MDM renamed /Modem/EN_V_3V8_MDM
- net /Modem/V_3V3_MDM_RAW renamed /Modem/V_3V8_MDM_RAW
- net /Power/V_OUT renamed /Power/V_3V8_OUT
- C209 pad 1: /Power/V_SYS -> /Power/V_IN
- C210 pad 1: /Power/V_SYS -> /Power/V_IN
- C503 pad 1: /Modem/V_3V3_MDM -> /Modem/V_BAT_RF
- C503 pad 2: GND -> Net-(C503-Pad2)
- C504 pad 1: /Modem/V_3V3_MDM -> /Modem/V_BAT_BB
- C504 pad 2: GND -> Net-(C504-Pad2)
- C506 pad 1: /Modem/V_3V3_MDM -> /Modem/V_BAT_RF
- C508 pad 1: /Modem/V_3V3_MDM -> /Modem/V_BAT_RF
- C509 pad 1: /Modem/PWRKEY -> /Modem/V_BAT_BB
- D503 pad 2: V_3V3 -> V_3V8
- FB501 pad 2: /Modem/V_3V3_MDM -> /Modem/V_BAT_RF
- J211 pad 2: V_3V3 -> V_3V8
- Q502 pad 2: V_3V3 -> V_3V8
- R219 pad 2: V_3V3 -> V_3V8
- R501 pad 1: V_3V3 -> V_3V8
- R509 pad 1: /Microcontroller/MDM_RI -> Net-(C503-Pad2)
- R509 pad 2: Net-(U501-B1) -> GND
- R510 pad 1: /Microcontroller/MDM_DCD -> Net-(C504-Pad2)
- R510 pad 2: Net-(U501-B2) -> GND
- R516 pad 1: Net-(U502-USIM_DATA) -> Net-(U502-USIM_RST)
- R516 pad 2: /Modem/SIM_DATA -> /Modem/SIM_RST
- R518 pad 1: Net-(U502-USIM_RST) -> /Modem/PSM_IND
- R518 pad 2: /Modem/SIM_RST -> GND
- U204 pad 10: /Power/V_SYS -> /Power/V_IN
- U204 pad 11: /Power/V_SYS -> /Power/V_IN
- U204 pad 14: unconnected-(U204-PG-Pad14) -> /Power/EN_V_3V3
- U301 pad 25: /Microcontroller/MDM_DCD -> Net-(U301-PB12)
- U301 pad 28: Net-(U301-PB15) -> unconnected-(U301-PB15-Pad28)
- U301 pad 29: /Microcontroller/MDM_RI -> unconnected-(U301-PA8-Pad29)
- U501 pad 1: /Modem/RI -> /Modem/PON_TRIG
- U501 pad 15: /Microcontroller/MDM_DTR -> unconnected-(U501-B5-Pad15)
- U501 pad 18: Net-(U501-B2) -> unconnected-(U501-B2-Pad18)
- U501 pad 20: Net-(U501-B1) -> /Microcontroller/MDM_PON
- U501 pad 3: /Modem/DCD -> unconnected-(U501-A2-Pad3)
- U501 pad 6: /Modem/DTR -> unconnected-(U501-A5-Pad6)
- U502 pad 1: unconnected-(U502-GPIO_1-Pad1) -> /Modem/PSM_IND
- U502 pad 13: Net-(U502-USIM_CLK) -> unconnected-(U502-RESERVED-Pad13)
- U502 pad 14: Net-(U502-USIM_DATA) -> unconnected-(U502-RESERVED-Pad14)
- U502 pad 15: Net-(U502-USIM_RST) -> /Modem/PWRKEY
- U502 pad 16: /Modem/V_1V8_SIM -> unconnected-(U502-RESERVED-Pad16)
- U502 pad 17: unconnected-(U502-ADC0-Pad17) -> /Modem/RESETn
- U502 pad 19: /Modem/V_3V3_MDM -> unconnected-(U502-GPIO6-Pad19)
- U502 pad 20: /Modem/V_3V3_MDM -> /Modem/STATUS
- U502 pad 21: /Modem/V_1V8_MDM -> /Modem/NET_STATUS
- U502 pad 22: GND -> unconnected-(U502-GPIO7-Pad22)
- U502 pad 23: GND -> unconnected-(U502-GPIO8-Pad23)
- U502 pad 24: GND -> unconnected-(U502-ADC0-Pad24)
- U502 pad 25: GND -> unconnected-(U502-GPIO9-Pad25)
- U502 pad 26: /Antennas/ANT -> unconnected-(U502-GPIO10-Pad26)
- U502 pad 27: GND -> unconnected-(U502-GPIO11-Pad27)
- U502 pad 28: GND -> unconnected-(U502-GPIO12-Pad28)
- U502 pad 29: unconnected-(U502-RSVD-Pad29) -> /Modem/V_1V8_MDM
- U502 pad 3: unconnected-(U502-PCM_CLK-Pad3) -> GND
- U502 pad 30: GND -> unconnected-(U502-MAIN_DTR-Pad30)
- U502 pad 32: unconnected-(U502-ANT_GNSS-Pad32) -> /Modem/V_BAT_BB
- U502 pad 33: unconnected-(U502-GPIO_4-Pad33) -> /Modem/V_BAT_BB
- U502 pad 34: unconnected-(U502-PCM_DOUT-Pad34) -> /Modem/TXD
- U502 pad 35: unconnected-(U502-PCM_SYNC-Pad35) -> /Modem/RXD
- U502 pad 36: unconnected-(U502-GNSS_TXD-Pad36) -> /Modem/CTS
- U502 pad 37: unconnected-(U502-I2C_SCL-Pad37) -> /Modem/RTS
- U502 pad 38: /Modem/RTS -> unconnected-(U502-MAIN_DCD-Pad38)
- U502 pad 39: /Modem/CTS -> unconnected-(U502-MAIN_RI-Pad39)
- U502 pad 42: unconnected-(U502-USBPHY_3P3-Pad42) -> /Modem/SIM_DET
- U502 pad 43: GND -> /Modem/V_1V8_SIM
- U502 pad 44: /Modem/SIM_DET -> Net-(U502-USIM_RST)
- U502 pad 45: /Modem/RESETn -> Net-(U502-USIM_DATA)
- U502 pad 46: /Modem/PWRKEY -> Net-(U502-USIM_CLK)
- U502 pad 48: unconnected-(U502-RSVD-Pad48) -> GND
- U502 pad 50: unconnected-(U502-RSVD-Pad50) -> GND
- U502 pad 52: GND -> /Modem/V_BAT_RF
- U502 pad 53: GND -> /Modem/V_BAT_RF
- U502 pad 56: GND -> unconnected-(U502-ANT_WIFI-Pad56)
- U502 pad 59: unconnected-(U502-RSVD-Pad59) -> GND
- U502 pad 6: /Modem/RXD -> unconnected-(U502-GPIO3-Pad6)
- U502 pad 60: unconnected-(U502-DBG_TXD-Pad60) -> /Antennas/ANT
- U502 pad 61: unconnected-(U502-DBG_RXD-Pad61) -> GND
- U502 pad 62: /Modem/DTR -> GND
- U502 pad 65: GND -> unconnected-(U502-GPIO16-Pad65)
- U502 pad 66: GND -> unconnected-(U502-GPIO17-Pad66)
- U502 pad 67: unconnected-(U502-RSVD-Pad67) -> GND
- U502 pad 68: unconnected-(U502-RSVD-Pad68) -> GND
- U502 pad 69: unconnected-(U502-RSVD-Pad69) -> GND
- U502 pad 7: /Modem/TXD -> unconnected-(U502-GPIO4-Pad7)
- U502 pad 70: unconnected-(U502-RSVD-Pad70) -> GND
- U502 pad 71: unconnected-(U502-RSVD-Pad71) -> GND
- U502 pad 72: unconnected-(U502-PON_TRIG-Pad72) -> GND
- U502 pad 75: GND -> unconnected-(U502-USB_BOOT-Pad75)
- U502 pad 76: /Modem/RI -> unconnected-(U502-RESERVED-Pad76)
- U502 pad 78: /Modem/STATUS -> unconnected-(U502-RESERVED-Pad78)
- U502 pad 79: /Modem/NET_STATUS -> GND
- U502 pad 80: unconnected-(U502-RSVD-Pad80) -> GND
- U502 pad 81: unconnected-(U502-RSVD-Pad81) -> GND
- U502 pad 82: unconnected-(U502-RSVD-Pad82) -> GND
- U502 pad 84: GND -> unconnected-(U502-GRFC2-Pad84)
- U502 pad 85: GND -> unconnected-(U502-GPIO18-Pad85)
- U502 pad 86: GND -> unconnected-(U502-GPIO19-Pad86)
- U502 pad 88: GND -> unconnected-(U502-GPIO21-Pad88)
- U502 pad 90: /Modem/DCD -> GND
- U502 pad 91: unconnected-(U502-RSVD-Pad91) -> GND
Routing:
- net /Power/EN_V_3V3: track 0.00 -> 23.4 mm, vias 0 -> 2
- net /Modem/SIM_DET: track 22.1 -> 6.43 mm, vias 2 -> 0
- net V_3V8: track 0.00 -> 15.3 mm, vias 0 -> 8
- net /Modem/MDM_PWR_ON: track 16.2 -> 3.34 mm, vias 3 -> 2
- net /Modem/V_1V8_SIM: track 23.3 -> 10.9 mm
- net /Modem/PWRKEY: track 9.28 -> 0.00 mm
- net /Modem/SIM_RST: track 14.4 -> 5.37 mm, vias 2 -> 0
- net unconnected-(U501-B5-Pad15): track 0.00 -> 7.98 mm, vias 0 -> 1
- net /Microcontroller/MDM_DTR: track 7.98 -> 0.00 mm, vias 1 -> 0
- net /Modem/MDM_RESET: track 9.76 -> 1.85 mm, vias 3 -> 2
- net /Modem/SIM_DATA: track 13.9 -> 6.62 mm
- net /Modem/SIM_CLK: track 16.1 -> 8.86 mm, vias 0 -> 1
- net /Modem/RESETn: track 6.72 -> 0.00 mm
- net Net-(U502-USIM_RST): track 4.44 -> 0.00 mm
- net Net-(U502-USIM_DATA): track 4.31 -> 0.00 mm
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- added copper zone on F.Cu, net /Power/V_3V3_OUT
- added copper zone on F.Cu, net /Power/V_IN
- added copper zone on F.Cu, net V_3V8
- removed copper zone on F.Cu, net /Modem/V_3V3_MDM
- removed copper zone on F.Cu, net /Modem/V_3V8_MDM_RAW
Other:
- board text added: "NET"
- board text added: "PG"
- board text added: "PSM"
- board text added: "STAT1"
- board text added: "STAT2"
- board text added: "STATUS"
- board text added: "V_3V8"
